File: psu/psu.kicad_pcb (KiCad board)
At the start: 2 copper layers, 19 parts, among them J1 Conn_01x10_MountingPin, U1 LM723, U2 BDX53, U3 TL071, U4 BDX54

Commit message: Add files via upload
Parts:
- C1: value C -> 470p
- C2, C5: value C_Polarized -> 470u
- C3, C6: value C_Polarized -> 10u
- C4: value C -> 0.1u
- C7: value C -> 0.1
- R1: value R_US -> 10R
- R2: value R_US -> 220R
- R3, R4, R5: value R_US -> 10k
- R6: value R_US -> 33R
- RV1: value R_Potentiometer_Trim -> 470R
Connections:
- R3 pad 2: -15V -> Net-(R3-Pad2)
- R5 pad 2: -15V -> Net-(R3-Pad2)
- U3 pad 2: -15V -> Net-(R3-Pad2)
Routing:
- net Net-(R3-Pad2): track 0.00 -> 28.2 mm
- net -15V: track 87.4 -> 64.0 mm
- net Net-(C1-Pad2): track 12.1 -> 13.4 mm
Other:
- board outline added: 124.1 x 32 mm
