File: psu/psu.sch (KiCad schematic (older format))
At the start: 19 parts, among them J1 Conn_01x10_MountingPin, U1 LM723, U2 BDX53, U3 TL071, U4 BDX54

Commit message: Add files via upload
Parts:
- C1: value C -> 470p
- C2, C5: value C_Polarized -> 470u
- C3, C6: value C_Polarized -> 10u
- C4: value C -> 0.1u
- C7: value C -> 0.1
- R1: value R_US -> 10R
- R2: value R_US -> 220R
- R3, R4, R5: value R_US -> 10k
- R6: value R_US -> 33R
- RV1: value R_Potentiometer_Trim -> 470R
Connections:
- net -15V: no longer R3.2, R5.2, U3.2 (-)
- new net: R3.2, R5.2, U3.2 (-)
Changed lines of the file:
@@
 P 4050 2100
 F 0 "R1" V 3845 2100 50  0000 C CNN
-F 1 "R_US" V 3936 2100 50  0000 C CNN
+F 1 "10R" V 3936 2100 50  0000 C CNN
 F 2 "Resistor_THT:R_Axial_DIN0207_L6.3mm_D2.5mm_P10.16mm_Horizontal" V 4090 2090 50  0001 C CNN
 F 3 "~" H 4050 2100 50  0001 C CNN
@@
 P 3750 2450
 F 0 "R2" V 3545 2450 50  0000 C CNN
-F 1 "R_US" V 3636 2450 50  0000 C CNN
+F 1 "220R" V 3636 2450 50  0000 C CNN
 F 2 "Resistor_THT:R_Axial_DIN0207_L6.3mm_D2.5mm_P10.16mm_Horizontal" V 3790 2440 50  0001 C CNN
 F 3 "~" H 3750 2450 50  0001 C CNN
@@
 P 3750 2950
 F 0 "RV1" H 3681 2996 50  0000 R CNN
-F 1 "R_Potentiometer_Trim" H 3681 2905 50  0000 R CNN
+F 1 "470R" H 3681 2905 50  0000 R CNN
 F 2 "Potentiometer_THT:Potentiometer_Bourns_3266Y_Vertical" H 3750 2950 50  0001 C CNN
 F 3 "~" H 3750 2950 50  0001 C CNN
@@
 P 3750 3400
 F 0 "R4" V 3545 3400 50  0000 C CNN
-F 1 "R_US" V 3636 3400 50  0000 C CNN
+F 1 "10k" V 3636 3400 50  0000 C CNN
 F 2 "Resistor_THT:R_Axial_DIN0207_L6.3mm_D2.5mm_P10.16mm_Horizontal" V 3790 3390 50  0001 C CNN
 F 3 "~" H 3750 3400 50  0001 C CNN
@@
 P 4350 1900
 F 0 "C1" V 4098 1900 50  0000 C CNN
-F 1 "C" V 4189 1900 50  0000 C CNN
+F 1 "470p" V 4189 1900 50  0000 C CNN
 F 2 "Capacitor_THT:C_Axial_L3.8mm_D2.6mm_P7.50mm_Horizontal" H 4388 1750 50  0001 C CNN
 F 3 "~" H 4350 1900 50  0001 C CNN
@@
 P 4450 3400
 F 0 "R5" V 4245 3400 50  0000 C CNN
-F 1 "R_US" V 4336 3400 50  0000 C CNN
+F 1 "10k" V 4336 3400 50  0000 C CNN
 F 2 "Resistor_THT:R_Axial_DIN0207_L6.3mm_D2.5mm_P10.16mm_Horizontal" V 4490 3390 50  0001 C CNN
 F 3 "~" H 4450 3400 50  0001 C CNN
@@
 P 6650 2100
 F 0 "C2" V 6905 2100 50  0000 C CNN
-F 1 "C_Polarized" V 6814 2100 50  0000 C CNN
+F 1 "470u" V 6814 2100 50  0000 C CNN
 F 2 "Capacitor_THT:CP_Radial_D16.0mm_P7.50mm" H 6688 1950 50  0001 C CNN
 F 3 "~" H 6650 2100 50  0001 C CNN
@@
 P 6650 2500
 F 0 "C3" V 6905 2500 50  0000 C CNN
-F 1 "C_Polarized" V 6814 2500 50  0000 C CNN
+F 1 "10u" V 6814 2500 50  0000 C CNN
 F 2 "Capacitor_THT:CP_Radial_D8.0mm_P5.00mm" H 6688 2350 50  0001 C CNN
 F 3 "~" H 6650 2500 50  0001 C CNN
@@
 P 6650 2850
 F 0 "C4" V 6398 2850 50  0000 C CNN
-F 1 "C" V 6489 2850 50  0000 C CNN
+F 1 "0.1u" V 6489 2850 50  0000 C CNN
 F 2 "Capacitor_THT:C_Axial_L3.8mm_D2.6mm_P7.50mm_Horizontal" H 6688 2700 50  0001 C CNN
 F 3 "~" H 6650 2850 50  0001 C CNN
@@
 P 6650 3100
 F 0 "R3" V 6445 3100 50  0000 C CNN
-F 1 "R_US" V 6536 3100 50  0000 C CNN
+F 1 "10k" V 6536 3100 50  0000 C CNN
 F 2 "Resistor_THT:R_Axial_DIN0207_L6.3mm_D2.5mm_P10.16mm_Horizontal" V 6690 3090 50  0001 C CNN
 F 3 "~" H 6650 3100 50  0001 C CNN
@@
 P 5650 4050
 F 0 "R6" V 5445 4050 50  0000 C CNN
-F 1 "R_US" V 5536 4050 50  0000 C CNN
+F 1 "33R" V 5536 4050 50  0000 C CNN
 F 2 "Resistor_THT:R_Axial_DIN0207_L6.3mm_D2.5mm_P10.16mm_Horizontal" V 5690 4040 50  0001 C CNN
 F 3 "~" H 5650 4050 50  0001 C CNN
@@
 P 4500 4000
 F 0 "C5" V 4755 4000 50  0000 C CNN
-F 1 "C_Polarized" V 4664 4000 50  0000 C CNN
+F 1 "470u" V 4664 4000 50  0000 C CNN
 F 2 "Capacitor_THT:CP_Radial_D16.0mm_P7.50mm" H 4538 3850 50  0001 C CNN
 F 3 "~" H 4500 4000 50  0001 C CNN
@@
 P 4500 4400
 F 0 "C6" V 4755 4400 50  0000 C CNN
-F 1 "C_Polarized" V 4664 4400 50  0000 C CNN
+F 1 "10u" V 4664 4400 50  0000 C CNN
 F 2 "Capacitor_THT:CP_Radial_D8.0mm_P5.00mm" H 4538 4250 50  0001 C CNN
 F 3 "~" H 4500 4400 50  0001 C CNN
@@
 P 4500 4750
 F 0 "C7" V 4248 4750 50  0000 C CNN
-F 1 "C" V 4339 4750 50  0000 C CNN
+F 1 "0.1" V 4339 4750 50  0000 C CNN
 F 2 "Capacitor_THT:C_Axial_L3.8mm_D2.6mm_P7.50mm_Horizontal" H 4538 4600 50  0001 C CNN
 F 3 "~" H 4500 4750 50  0001 C CNN
@@
 	6800 3100 6800 3000
 Wire Wire Line
-	6800 3000 5000 3000
-Wire Wire Line
 	4700 3000 4700 3400
-Connection ~ 5000 3000
-Wire Wire Line
-	5000 3000 4700 3000
 Connection ~ 4700 3400
 Wire Wire Line
@@
 Wire Wire Line
 	7900 2300 8500 2300
+Wire Wire Line
+	4700 3000 6800 3000
 $EndSCHEMATC
