File: vcaEG/vcaEG.sch (KiCad schematic (older format))
At the start: 33 parts, among them J1 Conn_01x10_MountingPin, Q1 BC307, Q2 BC237, Q3 BC237, Q4 BC237, Q5 BC237, SW1 SW_Rotary2x3, U1 TL071

Commit message: Add files via upload
Parts:
- added J2, J3: Conn_01x02_MountingPin, Connector_PinSocket_2.54mm:PinSocket_1x02_P2.54mm_Vertical, symbol Connector_Generic_MountingPin:Conn_01x02_MountingPin
- C1, C3: value C -> 0.01u
- C2: value C_Polarized -> 10u
- R1, R10, R12, R14, R3, R6, R7: value R_US -> 10k
- R11, R13, R15, R9: value R_US -> 22k
- R2: value R_US -> 560R
- R4: value R_US -> 3k3
- R5: value R_US -> 33k
- R8: value R_US -> 470R
- RV1, RV2: value R_Potentiometer -> 100k log
- SW1: footprint Connector_Molex:Molex_Mini-Fit_Jr_5566-08A_2x04_P4.20mm_Vertical -> Connector_PinSocket_2.54mm:PinSocket_1x04_P2.54mm_Vertical
Connections:
- net at R15.2, SW1.5, SW1.7: now also J3.1 (Pin_1)
- net at Q5.1 (C), R14.1, SW1.8: now also J3.2 (Pin_2)
- net at C3.1, SW1.4: now also J2.2 (Pin_2)
- net at J1.10 (Pin_10), SW1.1: now also J2.1 (Pin_1)
Changed lines of the file:
@@
 P 2500 1790
 F 0 "R1" H 2568 1836 50  0000 L CNN
-F 1 "R_US" H 2568 1745 50  0000 L CNN
+F 1 "10k" H 2568 1745 50  0000 L CNN
 F 2 "Resistor_THT:R_Axial_DIN0207_L6.3mm_D2.5mm_P10.16mm_Horizontal" V 2540 1780 50  0001 C CNN
 F 3 "~" H 2500 1790 50  0001 C CNN
@@
 P 2750 2090
 F 0 "C1" V 2498 2090 50  0000 C CNN
-F 1 "C" V 2589 2090 50  0000 C CNN
+F 1 "0.01u" V 2589 2090 50  0000 C CNN
 F 2 "Capacitor_THT:C_Axial_L5.1mm_D3.1mm_P10.00mm_Horizontal" H 2788 1940 50  0001 C CNN
 F 3 "~" H 2750 2090 50  0001 C CNN
@@
 P 7500 3140
 F 0 "C2" H 7618 3186 50  0000 L CNN
-F 1 "C_Polarized" H 7618 3095 50  0000 L CNN
+F 1 "10u" H 7618 3095 50  0000 L CNN
 F 2 "Capacitor_THT:CP_Axial_L10.0mm_D4.5mm_P15.00mm_Horizontal" H 7538 2990 50  0001 C CNN
 F 3 "~" H 7500 3140 50  0001 C CNN
@@
 P 6950 3140
 F 0 "RV1" H 6880 3186 50  0000 R CNN
-F 1 "R_Potentiometer" H 6880 3095 50  0000 R CNN
+F 1 "100k log" H 6880 3095 50  0000 R CNN
 F 2 "Potentiometer_THT:Potentiometer_Alps_RK163_Single_Horizontal" H 6950 3140 50  0001 C CNN
 F 3 "~" H 6950 3140 50  0001 C CNN
@@
 P 3450 1490
 F 0 "R6" V 3245 1490 50  0000 C CNN
-F 1 "R_US" V 3336 1490 50  0000 C CNN
+F 1 "10k" V 3336 1490 50  0000 C CNN
 F 2 "Resistor_THT:R_Axial_DIN0207_L6.3mm_D2.5mm_P10.16mm_Horizontal" V 3490 1480 50  0001 C CNN
 F 3 "~" H 3450 1490 50  0001 C CNN
@@
 P 3700 990
 F 0 "R4" H 3768 1036 50  0000 L CNN
-F 1 "R_US" H 3768 945 50  0000 L CNN
+F 1 "3k3" H 3768 945 50  0000 L CNN
 F 2 "Resistor_THT:R_Axial_DIN0207_L6.3mm_D2.5mm_P10.16mm_Horizontal" V 3740 980 50  0001 C CNN
 F 3 "~" H 3700 990 50  0001 C CNN
@@
 P 3700 540
 F 0 "R2" H 3768 586 50  0000 L CNN
-F 1 "R_US" H 3768 495 50  0000 L CNN
+F 1 "560R" H 3768 495 50  0000 L CNN
 F 2 "Resistor_THT:R_Axial_DIN0207_L6.3mm_D2.5mm_P10.16mm_Horizontal" V 3740 530 50  0001 C CNN
 F 3 "~" H 3700 540 50  0001 C CNN
@@
 P 4300 540
 F 0 "R3" H 4368 586 50  0000 L CNN
-F 1 "R_US" H 4368 495 50  0000 L CNN
+F 1 "10k" H 4368 495 50  0000 L CNN
 F 2 "Resistor_THT:R_Axial_DIN0207_L6.3mm_D2.5mm_P10.16mm_Horizontal" V 4340 530 50  0001 C CNN
 F 3 "~" H 4300 540 50  0001 C CNN
@@
 P 4600 1240
 F 0 "R5" V 4395 1240 50  0000 C CNN
-F 1 "R_US" V 4486 1240 50  0000 C CNN
+F 1 "33k" V 4486 1240 50  0000 C CNN
 F 2 "Resistor_THT:R_Axial_DIN0207_L6.3mm_D2.5mm_P10.16mm_Horizontal" V 4640 1230 50  0001 C CNN
 F 3 "~" H 4600 1240 50  0001 C CNN
@@
 P 5250 3640
 F 0 "R11" V 5045 3640 50  0000 C CNN
-F 1 "R_US" V 5136 3640 50  0000 C CNN
+F 1 "22k" V 5136 3640 50  0000 C CNN
 F 2 "Resistor_THT:R_Axial_DIN0207_L6.3mm_D2.5mm_P10.16mm_Horizontal" V 5290 3630 50  0001 C CNN
 F 3 "~" H 5250 3640 50  0001 C CNN
@@
 P 5650 2340
 F 0 "R9" H 5582 2294 50  0000 R CNN
-F 1 "R_US" H 5582 2385 50  0000 R CNN
+F 1 "22k" H 5582 2385 50  0000 R CNN
 F 2 "Resistor_THT:R_Axial_DIN0207_L6.3mm_D2.5mm_P10.16mm_Horizontal" V 5690 2330 50  0001 C CNN
 F 3 "~" H 5650 2340 50  0001 C CNN
@@
 P 5950 4390
 F 0 "R15" V 5745 4390 50  0000 C CNN
-F 1 "R_US" V 5836 4390 50  0000 C CNN
+F 1 "22k" V 5836 4390 50  0000 C CNN
 F 2 "Resistor_THT:R_Axial_DIN0207_L6.3mm_D2.5mm_P10.16mm_Horizontal" V 5990 4380 50  0001 C CNN
 F 3 "~" H 5950 4390 50  0001 C CNN
@@
 P 4600 3940
 F 0 "R14" H 4532 3894 50  0000 R CNN
-F 1 "R_US" H 4532 3985 50  0000 R CNN
+F 1 "10k" H 4532 3985 50  0000 R CNN
 F 2 "Resistor_THT:R_Axial_DIN0207_L6.3mm_D2.5mm_P10.16mm_Horizontal" V 4640 3930 50  0001 C CNN
 F 3 "~" H 4600 3940 50  0001 C CNN
@@
 P 3950 3940
 F 0 "R13" H 3882 3894 50  0000 R CNN
-F 1 "R_US" H 3882 3985 50  0000 R CNN
+F 1 "22k" H 3882 3985 50  0000 R CNN
 F 2 "Resistor_THT:R_Axial_DIN0207_L6.3mm_D2.5mm_P10.16mm_Horizontal" V 3990 3930 50  0001 C CNN
 F 3 "~" H 3950 3940 50  0001 C CNN
@@
 P 6550 3890
 F 0 "R12" H 6482 3844 50  0000 R CNN
-F 1 "R_US" H 6482 3935 50  0000 R CNN
+F 1 "10k" H 6482 3935 50  0000 R CNN
 F 2 "Resistor_THT:R_Axial_DIN0207_L6.3mm_D2.5mm_P10.16mm_Horizontal" V 6590 3880 50  0001 C CNN
 F 3 "~" H 6550 3890 50  0001 C CNN
@@
 P 7850 2840
 F 0 "R10" V 7645 2840 50  0000 C CNN
-F 1 "R_US" V 7736 2840 50  0000 C CNN
+F 1 "10k" V 7736 2840 50  0000 C CNN
 F 2 "Resistor_THT:R_Axial_DIN0207_L6.3mm_D2.5mm_P10.16mm_Horizontal" V 7890 2830 50  0001 C CNN
 F 3 "~" H 7850 2840 50  0001 C CNN
@@
 P 6550 2490
 F 0 "RV2" H 6480 2536 50  0000 R CNN
-F 1 "R_Potentiometer" H 6480 2445 50  0000 R CNN
+F 1 "100k log" H 6480 2445 50  0000 R CNN
 F 2 "Potentiometer_THT:Potentiometer_Alps_RK163_Single_Horizontal" H 6550 2490 50  0001 C CNN
 F 3 "~" H 6550 2490 50  0001 C CNN
@@
 P 6550 2090
 F 0 "R8" H 6482 2044 50  0000 R CNN
-F 1 "R_US" H 6482 2135 50  0000 R CNN
+F 1 "470R" H 6482 2135 50  0000 R CNN
 F 2 "Resistor_THT:R_Axial_DIN0207_L6.3mm_D2.5mm_P10.16mm_Horizontal" V 6590 2080 50  0001 C CNN
 F 3 "~" H 6550 2090 50  0001 C CNN
@@
 P 3050 3040
 F 0 "C3" H 2935 2994 50  0000 R CNN
-F 1 "C" H 2935 3085 50  0000 R CNN
+F 1 "0.01u" H 2935 3085 50  0000 R CNN
 F 2 "Capacitor_THT:C_Axial_L5.1mm_D3.1mm_P10.00mm_Horizontal" H 3088 2890 50  0001 C CNN
 F 3 "~" H 3050 3040 50  0001 C CNN
@@
 P 5650 1590
 F 0 "R7" H 5582 1544 50  0000 R CNN
-F 1 "R_US" H 5582 1635 50  0000 R CNN
+F 1 "10k" H 5582 1635 50  0000 R CNN
 F 2 "Resistor_THT:R_Axial_DIN0207_L6.3mm_D2.5mm_P10.16mm_Horizontal" V 5690 1580 50  0001 C CNN
 F 3 "~" H 5650 1590 50  0001 C CNN
@@
 F 0 "SW1" V 3049 3893 50  0000 L CNN
 F 1 "SW_Rotary2x3" V 3140 3893 50  0000 L CNN
-F 2 "Connector_Molex:Molex_Mini-Fit_Jr_5566-08A_2x04_P4.20mm_Vertical" H 2930 4050 50  0001 C CNN
+F 2 "Connector_PinSocket_2.54mm:PinSocket_1x04_P2.54mm_Vertical" H 2930 4050 50  0001 C CNN
 F 3 "http://cdn-reichelt.de/documents/datenblatt/C200/DS-Serie%23LOR.pdf" H 2930 4050 50  0001 C CNN
 	1    3050 3740
@@
 F 0 "SW1" H 5165 5305 50  0000 C CNN
 F 1 "SW_Rotary2x3" H 5165 5214 50  0000 C CNN
-F 2 "Connector_Molex:Molex_Mini-Fit_Jr_5566-08A_2x04_P4.20mm_Vertical" H 5080 5300 50  0001 C CNN
+F 2 "Connector_PinSocket_2.54mm:PinSocket_1x04_P2.54mm_Vertical" H 5080 5300 50  0001 C CNN
 F 3 "http://cdn-reichelt.de/documents/datenblatt/C200/DS-Serie%23LOR.pdf" H 5080 5300 50  0001 C CNN
 	2    5200 4990
@@
 $EndComp
 Wire Wire Line
-	3050 3190 3050 3440
+	3050 3190 3050 3330
 Wire Wire Line
 	4600 4290 4600 4090
@@
 	2810 820  3050 820
 Wire Wire Line
-	3270 4240 3270 6000
+	3270 4240 3270 4530
 Wire Wire Line
 	3270 6000 10000 6000
@@
 	7020 -470 7020 430
 $Comp
-L power:GND #PWR?
+L power:GND #PWR0116
 U 1 1 6460555D
 P 8330 230
-F 0 "#PWR?" H 8330 -20 50  0001 C CNN
+F 0 "#PWR0116" H 8330 -20 50  0001 C CNN
 F 1 "GND" H 8335 57  50  0000 C CNN
 F 2 "" H 8330 230 50  0001 C CNN
@@
 Wire Wire Line
 	8000 -70  8480 -70
+$Comp
+L Connector_Generic_MountingPin:Conn_01x02_MountingPin J2
+U 1 1 645729E1
+P 2255 3965
+F 0 "J2" H 2343 3787 50  0000 L CNN
+F 1 "Conn_01x02_MountingPin" H 2343 3878 50  0000 L CNN
+F 2 "Connector_PinSocket_2.54mm:PinSocket_1x02_P2.54mm_Vertical" H 2255 3965 50  0001 C CNN
+F 3 "~" H 2255 3965 50  0001 C CNN
+	1    2255 3965
+	-1   0    0    1
+$EndComp
+Wire Wire Line
+	2455 3865 2455 3330
+Wire Wire Line
+	2455 3330 3050 3330
+Connection ~ 3050 3330
+Wire Wire Line
+	3050 3330 3050 3440
+Wire Wire Line
+	3270 4530 2455 4530
+Wire Wire Line
+	2455 4530 2455 3965
+Connection ~ 3270 4530
+Wire Wire Line
+	3270 4530 3270 6000
+$Comp
+L Connector_Generic_MountingPin:Conn_01x02_MountingPin J3
+U 1 1 6457CCBE
+P 5360 5650
+F 0 "J3" V 5236 5730 50  0000 L CNN
+F 1 "Conn_01x02_MountingPin" V 5327 5730 50  0000 L CNN
+F 2 "Connector_PinSocket_2.54mm:PinSocket_1x02_P2.54mm_Vertical" H 5360 5650 50  0001 C CNN
+F 3 "~" H 5360 5650 50  0001 C CNN
+	1    5360 5650
+	0    1    1    0
+$EndComp
+Wire Wire Line
+	5360 5450 5700 5450
+Wire Wire Line
+	5700 5450 5700 5090
+Connection ~ 5700 5090
+Wire Wire Line
+	5260 5450 4800 5450
+Wire Wire Line
+	4800 5450 4800 4990
+Connection ~ 4800 4990
 $EndSCHEMATC
