File: vcf V2 avec pot/vcf.kicad_pcb (KiCad board)
At the start: 2 copper layers, 71 parts, among them J1 Conn_01x10_MountingPin, J2 Conn_01x05_MountingPin, Q1 BC237, Q10 BC307, Q11 BC237, Q2 BC237, Q3 BC237, Q4 BC237, Q5 BC237, Q6 BC237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

Commit message: Add files via upload
Parts:
- moved envelope1 45.5 mm to (43.9, 75.0), turned to 135 degrees
- moved resonance1 22.6 mm to (65.1, 53.8), turned to 135 degrees
- moved freq1 0.88 mm to (86.4, 32.6), turned to 135 degrees
Routing:
- net GND: track 248.1 -> 318.5 mm
- net Net-(R26-Pad2): track 165.2 -> 222.4 mm
- net Net-(R20-Pad1): track 12.8 -> 37.2 mm
- net -8V: track 146.3 -> 159.7 mm
- net Net-(J1-Pad9): track 71.6 -> 78.5 mm
- net Net-(R25-Pad2): track 33.4 -> 37.1 mm
