File: vcf V2 avec pot/vcf.sch (KiCad schematic (older format))
At the start: 71 parts, among them J1 Conn_01x10_MountingPin, J2 Conn_01x05_MountingPin, Q1 BC237, Q10 BC307, Q11 BC237, Q2 BC237, Q3 BC237, Q4 BC237, Q5 BC237, Q6 BC237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

Commit message: Add files via upload
Parts:
- C1, C6, C7: value C_Polarized -> 10u
- C2, C3, C4, C5: value C -> 0.1u
- C8: value C -> 0.47u
- C9: value C_Polarized -> 1u
- R1: value R_US -> 10k
- R10, R13, R7: value R_US -> 15k
- R11, R12, R20: value R_US -> 470R
- R14, R15, R16: value R_US -> 68k
- R17, R26: value R_US -> 100k
- R18: value R_US -> 22k
- R19, R8, R9: value R_US -> 2k7
- R2, R23: value R_US -> 2k2
- R21, R5: value R_US -> 4k7
- R22: value R_US -> 1k8
- R24, R25, R3: value R_US -> 150k
- R27, R31: value R_US -> 220k
- R28: value R_US -> 47k
- R29: value R_US -> 680k
- R30: value R_US -> 330k
- R4: value R_US -> 1k
- R6: value R_US -> 27k
- envelope1: value R_Potentiometer -> 100k lin
- freq1, resonance1: value R_Potentiometer -> 10k lin
- freqcalTRIMM1: value R_Potentiometer_Trim -> 100k
