File: vib+retrig+vca/vib+retrig+vca.sch (KiCad schematic (older format))
At the start: 49 parts, among them J1 Conn_01x10_MountingPin, J2 Conn_01x02_MountingPin, Q1 Q_NJFET_DSG, Q2 BC237, Q3 BC237, Q4 BC307, SW1 SW_SPDT, SW2 SW_SP3T, U1 TL072, U2 TL072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

Commit message: Add files via upload
Parts:
- added H2: MountingHole_Pad, MountingHole:MountingHole_2.2mm_M2_DIN965_Pad, symbol Mechanical:MountingHole_Pad
- C1, C6: value C -> 0.1u
- C2: value C -> 0.01u
- C3: value C_Polarized -> 10u
- Q1: value Q_NJFET_DSG -> 2N5163
- R1: value R_US -> 100R
- R10, R11: value R_US -> 330R
- R12, R20: value R_US -> 330k
- R13: value R_US -> 2k2
- R14, R19, R2, R24, R4, R8: value R_US -> 10k
- R15: value R_US -> 22k
- R16, R5: value R_US -> 100k
- R17, R22: value R_US -> 15k
- R18, R7: value R_US -> 3M3
- R21, R23, R9: value R_US -> 47k
- R3: value R_US -> 1M
- R6: value R_US -> 33k
- RV1: value R_Potentiometer_Trim -> 100k
- RV2, RV3: value R_Potentiometer -> 10k lin
- RV4: value R_Potentiometer -> 1M log
- RV5: value R_Potentiometer -> 100k lin
Connections:
- net at R14.2: now also H2.1
Changed lines of the file:
@@
 P 7000 1700
 F 0 "R6" V 6795 1700 50  0000 C CNN
-F 1 "R_US" V 6886 1700 50  0000 C CNN
+F 1 "33k" V 6886 1700 50  0000 C CNN
 F 2 "Resistor_THT:R_Axial_DIN0207_L6.3mm_D2.5mm_P10.16mm_Horizontal" V 7040 1690 50  0001 C CNN
 F 3 "~" H 7000 1700 50  0001 C CNN
@@
 P 9750 2150
 F 0 "C3" V 10005 2150 50  0000 C CNN
-F 1 "C_Polarized" V 9914 2150 50  0000 C CNN
+F 1 "10u" V 9914 2150 50  0000 C CNN
 F 2 "Capacitor_THT:CP_Axial_L10.0mm_D4.5mm_P15.00mm_Horizontal" H 9788 2000 50  0001 C CNN
 F 3 "~" H 9750 2150 50  0001 C CNN
@@
 P 3300 1650
 F 0 "C2" V 3048 1650 50  0000 C CNN
-F 1 "C" V 3139 1650 50  0000 C CNN
+F 1 "0.01u" V 3139 1650 50  0000 C CNN
 F 2 "Capacitor_THT:C_Axial_L3.8mm_D2.6mm_P7.50mm_Horizontal" H 3338 1500 50  0001 C CNN
 F 3 "~" H 3300 1650 50  0001 C CNN
@@
 P 950 1000
 F 0 "Q1" H 1141 1046 50  0000 L CNN
-F 1 "Q_NJFET_DSG" H 1141 955 50  0000 L CNN
+F 1 "2N5163" H 1141 955 50  0000 L CNN
 F 2 "Package_TO_SOT_THT:TO-92L_Wide" H 1150 1100 50  0001 C CNN
 F 3 "~" H 950 1000 50  0001 C CNN
@@
 P 1050 1550
 F 0 "R4" H 1118 1596 50  0000 L CNN
-F 1 "R_US" H 1118 1505 50  0000 L CNN
+F 1 "10k" H 1118 1505 50  0000 L CNN
 F 2 "Resistor_THT:R_Axial_DIN0207_L6.3mm_D2.5mm_P10.16mm_Horizontal" V 1090 1540 50  0001 C CNN
 F 3 "~" H 1050 1550 50  0001 C CNN
@@
 P 1900 1200
 F 0 "R2" H 1968 1246 50  0000 L CNN
-F 1 "R_US" H 1968 1155 50  0000 L CNN
+F 1 "10k" H 1968 1155 50  0000 L CNN
 F 2 "Resistor_THT:R_Axial_DIN0207_L6.3mm_D2.5mm_P10.16mm_Horizontal" V 1940 1190 50  0001 C CNN
 F 3 "~" H 1900 1200 50  0001 C CNN
@@
 P 2400 1900
 F 0 "R8" H 2468 1946 50  0000 L CNN
-F 1 "R_US" H 2468 1855 50  0000 L CNN
+F 1 "10k" H 2468 1855 50  0000 L CNN
 F 2 "Resistor_THT:R_Axial_DIN0207_L6.3mm_D2.5mm_P10.16mm_Horizontal" V 2440 1890 50  0001 C CNN
 F 3 "~" H 2400 1900 50  0001 C CNN
@@
 P 2050 1900
 F 0 "R7" H 2118 1946 50  0000 L CNN
-F 1 "R_US" H 2118 1855 50  0000 L CNN
+F 1 "3M3" H 2118 1855 50  0000 L CNN
 F 2 "Resistor_THT:R_Axial_DIN0207_L6.3mm_D2.5mm_P10.16mm_Horizontal" V 2090 1890 50  0001 C CNN
 F 3 "~" H 2050 1900 50  0001 C CNN
@@
 P 2750 1650
 F 0 "R5" V 2545 1650 50  0000 C CNN
-F 1 "R_US" V 2636 1650 50  0000 C CNN
+F 1 "100k" V 2636 1650 50  0000 C CNN
 F 2 "Resistor_THT:R_Axial_DIN0207_L6.3mm_D2.5mm_P10.16mm_Horizontal" V 2790 1640 50  0001 C CNN
 F 3 "~" H 2750 1650 50  0001 C CNN
@@
 P 2400 3300
 F 0 "R19" H 2468 3346 50  0000 L CNN
-F 1 "R_US" H 2468 3255 50  0000 L CNN
+F 1 "10k" H 2468 3255 50  0000 L CNN
 F 2 "Resistor_THT:R_Axial_DIN0207_L6.3mm_D2.5mm_P10.16mm_Horizontal" V 2440 3290 50  0001 C CNN
 F 3 "~" H 2400 3300 50  0001 C CNN
@@
 P 2050 3300
 F 0 "R18" H 2118 3346 50  0000 L CNN
-F 1 "R_US" H 2118 3255 50  0000 L CNN
+F 1 "3M3" H 2118 3255 50  0000 L CNN
 F 2 "Resistor_THT:R_Axial_DIN0207_L6.3mm_D2.5mm_P10.16mm_Horizontal" V 2090 3290 50  0001 C CNN
 F 3 "~" H 2050 3300 50  0001 C CNN
@@
 P 2750 3050
 F 0 "R16" V 2545 3050 50  0000 C CNN
-F 1 "R_US" V 2636 3050 50  0000 C CNN
+F 1 "100k" V 2636 3050 50  0000 C CNN
 F 2 "Resistor_THT:R_Axial_DIN0207_L6.3mm_D2.5mm_P10.16mm_Horizontal" V 2790 3040 50  0001 C CNN
 F 3 "~" H 2750 3050 50  0001 C CNN
@@
 P 4500 2000
 F 0 "R9" V 4295 2000 50  0000 C CNN
-F 1 "R_US" V 4386 2000 50  0000 C CNN
+F 1 "47k" V 4386 2000 50  0000 C CNN
 F 2 "Resistor_THT:R_Axial_DIN0207_L6.3mm_D2.5mm_P10.16mm_Horizontal" V 4540 1990 50  0001 C CNN
 F 3 "~" H 4500 2000 50  0001 C CNN
@@
 P 4150 3000
 F 0 "R15" H 4218 3046 50  0000 L CNN
-F 1 "R_US" H 4218 2955 50  0000 L CNN
+F 1 "22k" H 4218 2955 50  0000 L CNN
 F 2 "Resistor_THT:R_Axial_DIN0207_L6.3mm_D2.5mm_P10.16mm_Horizontal" V 4190 2990 50  0001 C CNN
 F 3 "~" H 4150 3000 50  0001 C CNN
@@
 P 1450 750
 F 0 "C1" V 1198 750 50  0000 C CNN
-F 1 "C" V 1289 750 50  0000 C CNN
+F 1 "0.1u" V 1289 750 50  0000 C CNN
 F 2 "Capacitor_THT:C_Axial_L3.8mm_D2.6mm_P7.50mm_Horizontal" H 1488 600 50  0001 C CNN
 F 3 "~" H 1450 750 50  0001 C CNN
@@
 P 2350 5150
 F 0 "R20" H 2418 5196 50  0000 L CNN
-F 1 "R_US" H 2418 5105 50  0000 L CNN
+F 1 "330k" H 2418 5105 50  0000 L CNN
 F 2 "Resistor_THT:R_Axial_DIN0207_L6.3mm_D2.5mm_P10.16mm_Horizontal" V 2390 5140 50  0001 C CNN
 F 3 "~" H 2350 5150 50  0001 C CNN
@@
 P 2700 5150
 F 0 "R21" H 2768 5196 50  0000 L CNN
-F 1 "R_US" H 2768 5105 50  0000 L CNN
+F 1 "47k" H 2768 5105 50  0000 L CNN
 F 2 "Resistor_THT:R_Axial_DIN0207_L6.3mm_D2.5mm_P10.16mm_Horizontal" V 2740 5140 50  0001 C CNN
 F 3 "~" H 2700 5150 50  0001 C CNN
@@
 P 3050 5150
 F 0 "RV4" H 2980 5196 50  0000 R CNN
-F 1 "R_Potentiometer" H 2980 5105 50  0000 R CNN
+F 1 "1M log" H 2980 5105 50  0000 R CNN
 F 2 "Potentiometer_THT:Potentiometer_Alps_RK163_Single_Horizontal" H 3050 5150 50  0001 C CNN
 F 3 "~" H 3050 5150 50  0001 C CNN
@@
 P 1800 6150
 F 0 "R22" V 1595 6150 50  0000 C CNN
-F 1 "R_US" V 1686 6150 50  0000 C CNN
+F 1 "15k" V 1686 6150 50  0000 C CNN
 F 2 "Resistor_THT:R_Axial_DIN0207_L6.3mm_D2.5mm_P10.16mm_Horizontal" V 1840 6140 50  0001 C CNN
 F 3 "~" H 1800 6150 50  0001 C CNN
@@
 P 2700 6150
 F 0 "R23" V 2495 6150 50  0000 C CNN
-F 1 "R_US" V 2586 6150 50  0000 C CNN
+F 1 "47k" V 2586 6150 50  0000 C CNN
 F 2 "Resistor_THT:R_Axial_DIN0207_L6.3mm_D2.5mm_P10.16mm_Horizontal" V 2740 6140 50  0001 C CNN
 F 3 "~" H 2700 6150 50  0001 C CNN
@@
 P 2200 6550
 F 0 "R24" V 1995 6550 50  0000 C CNN
-F 1 "R_US" V 2086 6550 50  0000 C CNN
+F 1 "10k" V 2086 6550 50  0000 C CNN
 F 2 "Resistor_THT:R_Axial_DIN0207_L6.3mm_D2.5mm_P10.16mm_Horizontal" V 2240 6540 50  0001 C CNN
 F 3 "~" H 2200 6550 50  0001 C CNN
@@
 P 4050 5400
 F 0 "C6" V 3798 5400 50  0000 C CNN
-F 1 "C" V 3889 5400 50  0000 C CNN
+F 1 "0.1u" V 3889 5400 50  0000 C CNN
 F 2 "Capacitor_THT:C_Axial_L3.8mm_D2.6mm_P7.50mm_Horizontal" H 4088 5250 50  0001 C CNN
 F 3 "~" H 4050 5400 50  0001 C CNN
@@
 P 3050 7400
 F 0 "RV5" H 2980 7446 50  0000 R CNN
-F 1 "R_Potentiometer" H 2980 7355 50  0000 R CNN
+F 1 "100k lin" H 2980 7355 50  0000 R CNN
 F 2 "Potentiometer_THT:Potentiometer_Alps_RK163_Single_Horizontal" H 3050 7400 50  0001 C CNN
 F 3 "~" H 3050 7400 50  0001 C CNN
@@
 P 7000 1200
 F 0 "R3" V 6795 1200 50  0000 C CNN
-F 1 "R_US" V 6886 1200 50  0000 C CNN
+F 1 "1M" V 6886 1200 50  0000 C CNN
 F 2 "Resistor_THT:R_Axial_DIN0207_L6.3mm_D2.5mm_P10.16mm_Horizontal" V 7040 1190 50  0001 C CNN
 F 3 "~" H 7000 1200 50  0001 C CNN
@@
 P 7200 2450
 F 0 "R10" V 6995 2450 50  0000 C CNN
-F 1 "R_US" V 7086 2450 50  0000 C CNN
+F 1 "330R" V 7086 2450 50  0000 C CNN
 F 2 "Resistor_THT:R_Axial_DIN0207_L6.3mm_D2.5mm_P10.16mm_Horizontal" V 7240 2440 50  0001 C CNN
 F 3 "~" H 7200 2450 50  0001 C CNN
@@
 P 7400 2450
 F 0 "R11" V 7195 2450 50  0000 C CNN
-F 1 "R_US" V 7286 2450 50  0000 C CNN
+F 1 "330R" V 7286 2450 50  0000 C CNN
 F 2 "Resistor_THT:R_Axial_DIN0207_L6.3mm_D2.5mm_P10.16mm_Horizontal" V 7440 2440 50  0001 C CNN
 F 3 "~" H 7400 2450 50  0001 C CNN
@@
 P 8350 2450
 F 0 "R12" V 8145 2450 50  0000 C CNN
-F 1 "R_US" V 8236 2450 50  0000 C CNN
+F 1 "330k" V 8236 2450 50  0000 C CNN
 F 2 "Resistor_THT:R_Axial_DIN0207_L6.3mm_D2.5mm_P10.16mm_Horizontal" V 8390 2440 50  0001 C CNN
 F 3 "~" H 8350 2450 50  0001 C CNN
@@
 P 9250 950
 F 0 "R1" V 9045 950 50  0000 C CNN
-F 1 "R_US" V 9136 950 50  0000 C CNN
+F 1 "100R" V 9136 950 50  0000 C CNN
 F 2 "Resistor_THT:R_Axial_DIN0207_L6.3mm_D2.5mm_P10.16mm_Horizontal" V 9290 940 50  0001 C CNN
 F 3 "~" H 9250 950 50  0001 C CNN
@@
 P 9250 2500
 F 0 "R13" V 9045 2500 50  0000 C CNN
-F 1 "R_US" V 9136 2500 50  0000 C CNN
+F 1 "2k2" V 9136 2500 50  0000 C CNN
 F 2 "Resistor_THT:R_Axial_DIN0207_L6.3mm_D2.5mm_P10.16mm_Horizontal" V 9290 2490 50  0001 C CNN
 F 3 "~" H 9250 2500 50  0001 C CNN
@@
 P 10150 2400
 F 0 "RV2" H 10080 2446 50  0000 R CNN
-F 1 "R_Potentiometer" H 10080 2355 50  0000 R CNN
+F 1 "10k lin" H 10080 2355 50  0000 R CNN
 F 2 "Potentiometer_THT:Potentiometer_Alps_RK163_Single_Horizontal" H 10150 2400 50  0001 C CNN
 F 3 "~" H 10150 2400 50  0001 C CNN
@@
 P 10500 2800
 F 0 "RV3" H 10430 2846 50  0000 R CNN
-F 1 "R_Potentiometer" H 10430 2755 50  0000 R CNN
+F 1 "10k lin" H 10430 2755 50  0000 R CNN
 F 2 "Potentiometer_THT:Potentiometer_Alps_RK163_Single_Horizontal" H 10500 2800 50  0001 C CNN
 F 3 "~" H 10500 2800 50  0001 C CNN
@@
 P 6450 1200
 F 0 "RV1" H 6381 1246 50  0000 R CNN
-F 1 "R_Potentiometer_Trim" H 6381 1155 50  0000 R CNN
+F 1 "100k" H 6381 1155 50  0000 R CNN
 F 2 "Potentiometer_THT:Potentiometer_Bourns_3266Y_Vertical" H 6450 1200 50  0001 C CNN
 F 3 "~" H 6450 1200 50  0001 C CNN
@@
 P 7300 3250
 F 0 "R17" V 7095 3250 50  0000 C CNN
-F 1 "R_US" V 7186 3250 50  0000 C CNN
+F 1 "15k" V 7186 3250 50  0000 C CNN
 F 2 "Resistor_THT:R_Axial_DIN0207_L6.3mm_D2.5mm_P10.16mm_Horizontal" V 7340 3240 50  0001 C CNN
 F 3 "~" H 7300 3250 50  0001 C CNN
@@
 P 10850 2550
 F 0 "R14" V 10645 2550 50  0000 C CNN
-F 1 "R_US" V 10736 2550 50  0000 C CNN
+F 1 "10k" V 10736 2550 50  0000 C CNN
 F 2 "Resistor_THT:R_Axial_DIN0207_L6.3mm_D2.5mm_P10.16mm_Horizontal" V 10890 2540 50  0001 C CNN
 F 3 "~" H 10850 2550 50  0001 C CNN
@@
 Wire Wire Line
 	2400 2050 2400 2100
+$Comp
+L Mechanical:MountingHole_Pad H2
+U 1 1 645326E4
+P 10850 2160
+F 0 "H2" H 10950 2209 50  0000 L CNN
+F 1 "MountingHole_Pad" H 10950 2118 50  0000 L CNN
+F 2 "MountingHole:MountingHole_2.2mm_M2_DIN965_Pad" H 10850 2160 50  0001 C CNN
+F 3 "~" H 10850 2160 50  0001 C CNN
+	1    10850 2160
+	1    0    0    -1
+$EndComp
+Wire Wire Line
+	10850 2260 10850 2400
 $EndSCHEMATC
